Commit message: [UPD] sdf to urdf

File: demo_common/demo_description/urdf/closed_link.urdf.xacro (robot description, xacro)
@@ -86,4 +86,32 @@
       <origin xyz="2 0 0" rpy="0 0 ${-M_PI/2}"/>
     </joint>
+    <gazebo>
+        <joint name='close_joint' type='continuous'>
+            <child>link_A</child>
+            <parent>link_D</parent>
+            <axis>
+                <xyz>0 0 1</xyz>
+                <limit>
+                    <lower>-1e+16</lower>
+                    <upper>1e+16</upper>
+                </limit>
+                <dynamics>
+                    <spring_reference>0</spring_reference>
+                    <spring_stiffness>0</spring_stiffness>
+                </dynamics>
+                <use_parent_model_frame>1</use_parent_model_frame>
+            </axis>
+        </joint>
+    </gazebo>
+    <!-- gazebo_ros_control plugins -->
+    <plugin name="gazebo_ros_control" filename="libgazebo_ros_control.so">
+      <robotNamespace>demo_model</robotNamespace>
+      <robotSimType>gazebo_ros_control/DefaultRobotHWSim</robotSimType>
+      <legacyModeNS>true</legacyModeNS>
+    </plugin>
+    <plugin name="joint_state_publisher" filename="libgazebo_ros_joint_state_publisher.so">
+      <robotNamespace>demo_model</robotNamespace>
+      <jointName>base_link_to_link_A, link_A_to_link_B, link_B_to_link_C, link_C_to_link_D, close_joint</jointName>
+    </plugin>
   </xacro:macro>
 </robot>

Commit message: [UPD] gazebo visualize

File: demo_common/demo_description/urdf/closed_link.urdf.xacro (robot description, xacro)
@@ -4,5 +4,15 @@
   <xacro:include filename="$(find demo_description)/urdf/closed_link.transmission.xacro"/>
   <xacro:macro name="closed_link" params="parent *joint_origin">
+    <joint name="${parent}_to_link_A" type="fixed">
+      <parent link="${parent}"/>
+      <child link="link_A"/>
+      <xacro:insert_block name="joint_origin"/>
+    </joint>
     <link name="link_A">
+      <inertial>
+        <origin xyz="1 0 0" rpy="0 0 0"/>
+        <mass value="0.5"/>
+        <inertia ixx="0.01" ixy="0.0" ixz="0.0" iyy="0.17" iyz="0.0" izz="0.17"/>
+      </inertial>
       <visual>
         <origin xyz="1 0 0" rpy="0 0 0"/>
@@ -14,9 +24,23 @@
         <origin xyz="1 0 0" rpy="0 0 0"/>
         <geometry>
-          <box size="2. 0.1 0.1"/>
+          <box size="2.0 0.1 0.1"/>
         </geometry>
       </collision>
     </link>
+    <joint name="link_A_to_link_B" type="revolute">
+      <axis xyz="0 0 1"/>
+      <limit lower="${-M_PI/4}" upper="${M_PI/4}" effort="100.0" velocity="${M_PI}"/>
+      <dynamics damping="0.1"/>
+      <parent link="link_A"/>
+      <child link="link_B"/>
+      <origin xyz="2 0 0" rpy="0 0 ${-M_PI/2}"/>
+    </joint>
+    <xacro:effort_trans joint="link_A_to_link_B"/>
     <link name="link_B">
+      <inertial>
+        <origin xyz="1 0 0" rpy="0 0 0"/>
+        <mass value="0.5"/>
+        <inertia ixx="0.01" ixy="0.0" ixz="0.0" iyy="0.17" iyz="0.0" izz="0.17"/>
+      </inertial>
       <visual>
         <origin xyz="1 0 0" rpy="0 0 0"/>
@@ -28,9 +52,20 @@
         <origin xyz="1 0 0" rpy="0 0 0"/>
         <geometry>
-          <box size="2. 0.1 0.1"/>
+          <box size="2.0 0.1 0.1"/>
         </geometry>
       </collision>
     </link>
+    <!-- <joint name="link_B_to_link_C" type="continuous">
+      <axis xyz="0 0 1"/>
+      <parent link="link_B"/>
+      <child link="link_C"/>
+      <origin xyz="2 0 0" rpy="0 0 ${-M_PI/2}"/>
+    </joint>
     <link name="link_C">
+      <inertial>
+        <origin xyz="1 0 0" rpy="0 0 0"/>
+        <mass value="0.5"/>
+        <inertia ixx="0.01" ixy="0.0" ixz="0.0" iyy="0.17" iyz="0.0" izz="0.17"/>
+      </inertial>
       <visual>
         <origin xyz="1 0 0" rpy="0 0 0"/>
@@ -42,9 +77,20 @@
         <origin xyz="1 0 0" rpy="0 0 0"/>
         <geometry>
-          <box size="2. 0.1 0.1"/>
+          <box size="2.0 0.1 0.1"/>
         </geometry>
       </collision>
     </link>
+    <joint name="link_C_to_link_D" type="continuous">
+      <axis xyz="0 0 1"/>
+      <parent link="link_C"/>
+      <child link="link_D"/>
+      <origin xyz="2 0 0" rpy="0 0 ${-M_PI/2}"/>
+    </joint>
     <link name="link_D">
+      <inertial>
+        <origin xyz="1 0 0" rpy="0 0 0"/>
+        <mass value="0.5"/>
+        <inertia ixx="0.01" ixy="0.0" ixz="0.0" iyy="0.17" iyz="0.0" izz="0.17"/>
+      </inertial>
       <visual>
         <origin xyz="1 0 0" rpy="0 0 0"/>
@@ -56,34 +102,8 @@
         <origin xyz="1 0 0" rpy="0 0 0"/>
         <geometry>
-          <box size="2. 0.1 0.1"/>
+          <box size="2.0 0.1 0.1"/>
         </geometry>
       </collision>
-    </link>
-    <joint name="${parent}_to_link_A" type="fixed">
-      <parent link="${parent}"/>
-      <child link="link_A"/>
-      <xacro:insert_block name="joint_origin"/>
-    </joint>
-    <joint name="link_A_to_link_B" type="revolute">
-      <axis xyz="0 0 1"/>
-      <limit lower="${-M_PI/4}" upper="${M_PI/4}" effort="100.0" velocity="${M_PI}"/>
-      <dynamics damping="0.1"/>
-      <parent link="link_A"/>
-      <child link="link_B"/>
-      <origin xyz="2 0 0" rpy="0 0 ${-M_PI/2}"/>
-    </joint>
-    <xacro:effort_trans joint="link_A_to_link_B"/>
-    <joint name="link_B_to_link_C" type="continuous">
-      <axis xyz="0 0 1"/>
-      <parent link="link_B"/>
-      <child link="link_C"/>
-      <origin xyz="2 0 0" rpy="0 0 ${-M_PI/2}"/>
-    </joint>
-    <joint name="link_C_to_link_D" type="continuous">
-      <axis xyz="0 0 1"/>
-      <parent link="link_C"/>
-      <child link="link_D"/>
-      <origin xyz="2 0 0" rpy="0 0 ${-M_PI/2}"/>
-    </joint>
+    </link> -->
     <gazebo>
         <joint name='close_joint' type='continuous'>
@@ -112,5 +132,5 @@
     <plugin name="joint_state_publisher" filename="libgazebo_ros_joint_state_publisher.so">
       <robotNamespace>demo_model</robotNamespace>
-      <jointName>base_link_to_link_A, link_A_to_link_B, link_B_to_link_C, link_C_to_link_D, close_joint</jointName>
+      <jointName>base_link_to_link_A, link_A_to_link_B</jointName>
     </plugin>
   </xacro:macro>
