Commit message: [ADD] initial setup for demo bringup and gazebo control packages

File: demo_description/urdf/closed_link.urdf.xacro (robot description, xacro)
@@ -4,6 +4,6 @@
   <xacro:include filename="$(find demo_description)/urdf/closed_link.transmission.xacro"/>
   <xacro:macro name="closed_link" params="parent *joint_origin">
-    <joint name="${parent}_to_link_A" type="fixed">
-      <parent link="${parent}"/>
+    <joint name="base_link_to_link_A" type="fixed">
+      <parent link="base_link"/>
       <child link="link_A"/>
       <xacro:insert_block name="joint_origin"/>
@@ -36,5 +36,5 @@
       <origin xyz="2 0 0" rpy="0 0 ${-M_PI/2}"/>
     </joint>
-    <xacro:effort_trans joint="link_A_to_link_B"/>
+    <xacro:position_trans joint="link_A_to_link_B"/>
     <link name="link_B">
       <inertial>
@@ -56,5 +56,5 @@
       </collision>
     </link>
-    <!-- <joint name="link_B_to_link_C" type="continuous">
+    <joint name="link_B_to_link_C" type="continuous">
       <axis xyz="0 0 1"/>
       <parent link="link_B"/>
@@ -105,33 +105,38 @@
         </geometry>
       </collision>
-    </link> -->
+    </link>
     <gazebo>
-        <joint name='close_joint' type='continuous'>
-            <child>link_A</child>
-            <parent>link_D</parent>
-            <axis>
-                <xyz>0 0 1</xyz>
-                <limit>
-                    <lower>-1e+16</lower>
-                    <upper>1e+16</upper>
-                </limit>
-                <dynamics>
-                    <spring_reference>0</spring_reference>
-                    <spring_stiffness>0</spring_stiffness>
-                </dynamics>
-                <use_parent_model_frame>1</use_parent_model_frame>
-            </axis>
-        </joint>
+      <joint name='close_joint' type='revolute'>
+        <child>link_A</child>
+        <parent>link_D</parent>
+        <axis>
+          <xyz>0 0 1</xyz>
+          <limit>
+            <lower>-1e+16</lower>
+            <upper>1e+16</upper>
+          </limit>
+          <dynamics>
+            <spring_reference>0</spring_reference>
+            <spring_stiffness>0</spring_stiffness>
+          </dynamics>
+          <use_parent_model_frame>1</use_parent_model_frame>
+        </axis>
+      </joint>
     </gazebo>
     <!-- gazebo_ros_control plugins -->
-    <plugin name="gazebo_ros_control" filename="libgazebo_ros_control.so">
-      <robotNamespace>demo_model</robotNamespace>
-      <robotSimType>gazebo_ros_control/DefaultRobotHWSim</robotSimType>
-      <legacyModeNS>true</legacyModeNS>
-    </plugin>
-    <plugin name="joint_state_publisher" filename="libgazebo_ros_joint_state_publisher.so">
-      <robotNamespace>demo_model</robotNamespace>
-      <jointName>base_link_to_link_A, link_A_to_link_B</jointName>
-    </plugin>
+    <gazebo>
+      <plugin name="gazebo_ros_control" filename="libgazebo_ros_control.so">
+        <robotNamespace>demo_model</robotNamespace>
+        <robotSimType>gazebo_ros_control/DefaultRobotHWSim</robotSimType>
+        <legacyModeNS>true</legacyModeNS>
+      </plugin>
+    </gazebo>
+    <gazebo>
+      <plugin name="joint_state_publisher" filename="libgazebo_ros_joint_state_publisher.so">
+        <robotNamespace>demo_model</robotNamespace>
+        <jointName>link_A_to_link_B, link_B_to_link_C, link_C_to_link_D</jointName>
+        <updateRate>50.0</updateRate>
+      </plugin>
+    </gazebo>
   </xacro:macro>
 </robot>

Commit message: [UPD] revolute to continous link_A_to_link_B

File: demo_description/urdf/closed_link.urdf.xacro (robot description, xacro)
@@ -28,5 +28,5 @@
       </collision>
     </link>
-    <joint name="link_A_to_link_B" type="revolute">
+    <joint name="link_A_to_link_B" type="continuous">
       <axis xyz="0 0 1"/>
       <limit lower="${-M_PI/4}" upper="${M_PI/4}" effort="100.0" velocity="${M_PI}"/>
